File: climate_control_niva_travel.kicad_sch (KiCad schematic)
At the start: 106 parts, among them J1 Разъём к автомобилю 2x16 (32 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, SW1 Кнопка тактовая 6x6 без фикса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, SW2 Кнопка тактовая 6x6 без фикса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, SW3 Кнопка тактовая 6x6 без фикса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, SW4 Кнопка тактовая 6x6 без фикса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, SW5 Кнопка тактовая 6x6 без фикса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, SW6 Кнопка тактовая 6x6 без фикса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, U1 STM32F103RCT6, U2 DRV8871 H-мост, U3 DRV8871 H-мост, U4 DRV8871 H-мост, U5 DRV8871 H-мост, U6 MC78M05CDTG, U7 AMS1117-3.3, U8 MCP2562-E-SN

Commit message: add power protect
Parts:
- added C20: 1uF 25В, Capacitor_SMD:C_0805_2012Metric, symbol Device:C
- added D5: SMBJ5.0A / 5,6В, Diode_SMD:D_SMB, symbol Device:D_Zener
- added L1: Феррит/дроссель по входу +12В (помехи), Inductor_SMD:L_1210_3225Metric, symbol Device:L
Connections:
- net GND: now also C20.2, D5.2 (A)
- net V5_SENS: now also D5.1 (K)
- net VCC_12V: now also C20.1, L1.2; no longer D1.1 (K)
- net at D1.2 (A), J1.1 (Pin_1), J1.2 (Pin_2): now also D1.1 (K), L1.1

Commit message: update sheme, tests on spiceng
Parts:
- removed C1: 470uF 25В, Capacitor_SMD:CP_Elec_10x10.5, symbol Device:C
- removed C11: 100uF 25В, Capacitor_SMD:CP_Elec_8x10.5, symbol Device:C
- removed C12, C13, C14, C15, C16, C17, C18, C19, C2, C_CABIN, C_CND, C_FAN, C_FB1, C_FB2, C_FB3, C_FB4, C_ILL, C_NRST, C_OZH, C_SOL, C_TEMP: 100nF, Capacitor_SMD:C_0603_1608Metric, symbol Device:C
- removed C20: 1uF 25В, Capacitor_SMD:C_0805_2012Metric, symbol Device:C
- removed C3: 10uF 35В, Capacitor_SMD:C_0805_2012Metric, symbol Device:C
- removed C4: 10uF 10В, Capacitor_SMD:C_0805_2012Metric, symbol Device:C
- removed D1: SS54, Diode_SMD:D_SMA, symbol Device:D_Schottky
- removed D2: SMBJ15A TVS, Diode_SMD:D_SMB, symbol Device:D_Zener
- removed D3: 1N4148W, Diode_SMD:D_SOD-123, symbol Device:D
- removed D4: SS14, Diode_SMD:D_SMA, symbol Device:D_Schottky
- removed D5: SMBJ5.0A / 5,6В, Diode_SMD:D_SMB, symbol Device:D_Zener
- removed J1: Разъём к автомобилю 2x16 (32 конт.), Connector_PinHeader_2.54mm:PinHeader_2x16_P2.54mm_Horizontal, symbol Connector_Generic:Conn_02x16_Odd_Even
- removed J_DBG: SWD-отладка 1x04, Connector_PinHeader_2.54mm:PinHeader_1x04_P2.54mm_Vertical, symbol Connector_Generic:Conn_01x04
- removed J_POT: Внутр. коннектор потенциометра (2п, XH), Connector_JST:JST_XH_B2B-XH-A_1x02_P2.50mm_Vertical, symbol Connector_Generic:Conn_01x02
- removed J_SENS_FAN: Внутр. коннектор вентилятора продувки (2п, XH), Connector_JST:JST_XH_B2B-XH-A_1x02_P2.50mm_Vertical, symbol Connector_Generic:Conn_01x02
- removed J_SW: Внутр. коннектор галлетника (2п, XH), Connector_JST:JST_XH_B2B-XH-A_1x02_P2.50mm_Vertical, symbol Connector_Generic:Conn_01x02
- removed L1: Феррит/дроссель по входу +12В (помехи), Inductor_SMD:L_1210_3225Metric, symbol Device:L
- removed LED1, LED2, LED3, LED5, LED6: Индикатор зелёный 1206, LED_SMD:LED_1206_3216Metric, symbol Device:LED
- removed LED4: Индикатор янтарный 1206, LED_SMD:LED_1206_3216Metric, symbol Device:LED
- removed Q_AC_N: MMBT3904, Package_TO_SOT_SMD:SOT-23, symbol Device:Q_NPN
- removed Q_AC_P: MMBT3906, Package_TO_SOT_SMD:SOT-23, symbol Device:Q_PNP
- removed Q_FAN: BSS138, Package_TO_SOT_SMD:SOT-23, symbol Device:Q_NMOS
- removed Q_MFAN: AO3400, Package_TO_SOT_SMD:SOT-23, symbol Device:Q_NMOS
- removed RT1: NTC 10k B3435,, Resistor_THT:R_Axial_DIN0204_L3.6mm_D1.6mm_P7.62mm_Horizontal, symbol Device:Thermistor_NTC
- removed R_AC_1, R_AC_PU, R_CABIN_UP, R_CND_A, R_FAN_UP, R_FB1_A, R_FB2_A, R_FB3_A, R_FB4_A, R_ILL_B, R_MFAN_GD, R_NRST, R_OZH_PROT, R_OZH_UP, R_SOL_A, R_TEMP_UP: 10k, Resistor_SMD:R_0603_1608Metric, symbol Device:R
- removed R_AC_GD: 100k, Resistor_SMD:R_0603_1608Metric, symbol Device:R
- removed R_AC_SER, R_FAN_GATE, R_FAN_SER, R_LED1, R_LED2, R_LED3, R_LED4, R_LED5, R_LED6, R_MFAN_G: 1k, Resistor_SMD:R_0603_1608Metric, symbol Device:R
- removed R_BOOT: 10k BOOT0, Resistor_SMD:R_0603_1608Metric, symbol Device:R
- removed R_CND_B, R_FB1_B, R_FB2_B, R_FB3_B, R_FB4_B, R_SOL_B: 20k, Resistor_SMD:R_0603_1608Metric, symbol Device:R
- removed R_FAN_PU: 4.7k, Resistor_SMD:R_0603_1608Metric, symbol Device:R
- removed R_ILIM1, R_ILIM2, R_ILIM3, R_ILIM4: 33k, Resistor_SMD:R_0603_1608Metric, symbol Device:R
- removed R_ILL_A: 47k, Resistor_SMD:R_0603_1608Metric, symbol Device:R
- removed SW1, SW2, SW3, SW4, SW5, SW6: Кнопка тактовая 6x6 без фиксации, Button_Switch_THT:SW_Push_1P1T_NO_6x6mm_H7.0mm, symbol Switch:SW_Push
- removed U2, U3, U4, U5: DRV8871 H-мост, Package_SO:SOIC-8_3.9x4.9mm_P1.27mm, symbol Driver_Motor:DRV8871DDA
- removed U6: MC78M05CDTG, Package_TO_SOT_SMD:TO-252-3_TabPin2, symbol Regulator_Linear:LM78M05_TO252
- removed U7: AMS1117-3.3, Package_TO_SOT_SMD:SOT-223-3_TabPin2, symbol Regulator_Linear:AP1117-15
- removed U8: MCP2562-E-SN, Package_SO:SOIC-8_3.9x4.9mm_P1.27mm, symbol Interface_CAN_LIN:MCP2562-E-SN
- added C21: 100nF, symbol Device:C
- added J2: SWD-отладка 1x04, symbol Connector_Generic:Conn_01x04
- added R1: 10k, symbol Device:R
- added R2: 10k BOOT0, symbol Device:R
- C10, C7, C8, C9: footprint Capacitor_SMD:C_0603_1608Metric -> (none)
- C5, C6: footprint Capacitor_SMD:C_0805_2012Metric -> (none)
- FB1: footprint Inductor_SMD:L_0805_2012Metric -> (none)
- U1: footprint Package_QFP:LQFP-64_10x10mm_P0.5mm -> (none)
Connections:
- net GND: now also C21.2, J2.4 (Pin_4), R2.2
- net NTC_CABIN: no longer C10.1, FB1.2, U1.60 (BOOT0)
- net TEMP_SET_ADC: no longer U1.7 (NRST)
- net VCC_3V3: now also J2.1 (Pin_1), R1.1; no longer U1.13 (VDDA)
- net SWDIO: now reaches U1.46 (PA13)
- net SWDIO: now also J2.2 (Pin_2)
- net SWCLK: now reaches U1.49 (PA14)
- net SWCLK: now also J2.3 (Pin_3)
- new net BOOT0: R2.1, U1.60 (BOOT0)
- new net NRST: C21.1, R1.2, U1.7 (NRST)
- new net VDDA_3V3: C10.1, FB1.2, U1.13 (VDDA)
- no-connect marks 0 -> 13
Other:
- added sheet ACT (cc_10_act.kicad_sch)
- added sheet CAN (cc_02_can.kicad_sch)
- added sheet OUT (cc_09_out.kicad_sch)
- added sheet PWR (cc_03_pwr.kicad_sch)
- added sheet SEN_CABIN (cc_05_sen_cabin.kicad_sch)
- added sheet SEN_COND (cc_08_sen_cond.kicad_sch)
- added sheet SEN_HEAT (cc_06_sen_heat.kicad_sch)
- added sheet SEN_SOLAR (cc_07_sen_solar.kicad_sch)
- added sheet UI (cc_04_ui.kicad_sch)
- note removed: "ACT"
- note removed: "MAIN"
- note removed: "MCU"
- note removed: "OUT"
- note removed: "SEN_CABIN"
- note removed: "SEN_COND"
- note removed: "SEN_HEAT"
- note removed: "SEN_SOLAR"
- note removed: "UI"
- company: DIY / Climate Control Niva Travel -> (none)
- title: MAIN -> CONTROLLER

Commit message: авто трассировка почти готова
Parts:
- C10, C21, C7, C8, C9, FB1, J2, R1, U1: mirror (none) -> None
- C5, C6: value 10uF 6,3В -> 10uF; mirror (none) -> None
- R2: value 10k BOOT0 -> 10k; mirror (none) -> None
Connections:
- net AC_CTL is gone; now on net AC_REQ_OUT: U1.28 (PB2)
- net BOOT0 is gone; now on net AC_REQ_OUT: R2.1, U1.60 (BOOT0)
- net BTN_DEFROST_GLASS is gone; now on net AC_REQ_OUT: U1.33 (PB12)
- net BTN_DRY_GLASS is gone; now on net BTN_RECIRC: U1.36 (PB15)
- net BTN_FACE is gone; now on net AC_REQ_OUT: U1.34 (PB13)
- net BTN_FEET is gone; now on net BTN_AC: U1.35 (PB14)
- net CAN_RX is gone; now on net AC_REQ_OUT: U1.61 (PB8)
- net CAN_TX is gone; now on net AC_REQ_OUT: U1.62 (PB9)
- net COND_ADC is gone; now on net AC_REQ_OUT: U1.21 (PA5)
- net FAN_PWM_CTL is gone; now on net AC_REQ_OUT: U1.41 (PA8)
- net FAN_SEL_ADC is gone; now on net AC_REQ_OUT: U1.15 (PA1)
- net FB_M1 is gone; now on net AC_REQ_OUT: U1.22 (PA6)
- net FB_M2 is gone; now on net AC_REQ_OUT: U1.23 (PA7)
- net FB_M3 is gone; now on net AC_REQ_OUT: U1.26 (PB0)
- net GND is gone; now on net AC_REQ_OUT: C10.2, C21.2, C5.2, C6.2, C7.2, C8.2, C9.2, J2.4 (Pin_4), R2.2, U1.12 (VSSA), U1.18 (VSS), U1.31 (VSS), U1.47 (VSS), U1.63 (VSS)
- net M1_IN1 is gone; now on net AC_REQ_OUT: U1.57 (PB5)
- net M1_IN2 is gone; now on net AC_REQ_OUT: U1.58 (PB6)
- net M2_IN1 is gone; now on net AC_REQ_OUT: U1.42 (PA9)
- net M2_IN2 is gone; now on net AC_REQ_OUT: U1.43 (PA10)
- net M3_IN1 is gone; now on net AC_REQ_OUT: U1.44 (PA11)
- net M3_IN2 is gone; now on net AC_REQ_OUT: U1.45 (PA12)
- net NRST is gone; now on net AC_REQ_OUT: C21.1, R1.2, U1.7 (NRST)
- net NTC_CABIN is gone; now on net AC_REQ_OUT: U1.16 (PA2)
- net NTC_HEAT is gone; now on net AC_REQ_OUT: U1.17 (PA3)
- net SOLAR_ADC is gone; now on net AC_REQ_OUT: U1.20 (PA4)
- net SWCLK is gone; now on net AC_REQ_OUT: J2.3 (Pin_3), U1.49 (PA14)
- net SWDIO is gone; now on net AC_REQ_OUT: J2.2 (Pin_2), U1.46 (PA13)
- net VCC_3V3 is gone; now on net AC_REQ_OUT: C5.1, C6.1, C7.1, C8.1, C9.1, FB1.1, J2.1 (Pin_1), R1.1, U1.1 (VBAT), U1.19 (VDD), U1.32 (VDD), U1.48 (VDD), U1.64 (VDD)
- net VDDA_3V3 is gone; now on net AC_REQ_OUT: C10.1, FB1.2, U1.13 (VDDA)
- net AC_REQ_OUT: now also U1.10 (PC2), U1.29 (PB10), U1.30 (PB11), U1.4 (PC15), U1.56 (PB4)
- net BTN_AC: no longer U1.51 (PC10)
- net BTN_RECIRC: no longer U1.52 (PC11)
- net ILLUM_SENSE: now also U1.8 (PC0); no longer U1.5 (PD0)
- net LED_DEFROST_GLASS_DRV: now also U1.50 (PA15); no longer U1.37 (PC6)
- net LED_DRY_GLASS_DRV: now also U1.3 (PC14); no longer U1.40 (PC9)
- net LED_FACE_DRV: now also U1.55 (PB3); no longer U1.38 (PC7)
- net M_FAN_CTL: now also U1.11 (PC3); no longer U1.50 (PA15)
- net LED_AC_DRV: no longer names the net of U1.53 (PC12)
- net LED_FEET_DRV: no longer names the net of U1.39 (PC8)
- net LED_RECIRC_DRV: no longer names the net of U1.54 (PD2)
- no-connect marks 13 -> 0
Other:
- removed sheet ACT
- removed sheet CAN
- removed sheet OUT
- removed sheet PWR
- removed sheet SEN_CABIN
- removed sheet SEN_COND
- removed sheet SEN_HEAT
- removed sheet SEN_SOLAR
- removed sheet UI
- added sheet X_ACT (sheets/actuators.kicad_sch)
- added sheet X_BACKLIGHT (sheets/backlight.kicad_sch)
- added sheet X_CAN (sheets/can_bus.kicad_sch)
- added sheet X_OUT (sheets/power_outputs.kicad_sch)
- added sheet X_PWR (sheets/power_supply.kicad_sch)
- added sheet X_SEN_CABIN (sheets/cabin_sensor.kicad_sch)
- added sheet X_SEN_COND (sheets/condensate_sensor.kicad_sch)
- added sheet X_SEN_HEAT (sheets/heating_sensor.kicad_sch)
- added sheet X_SEN_SOLAR (sheets/solar_sensor.kicad_sch)
- added sheet X_UI (sheets/user_interface.kicad_sch)
- title: CONTROLLER -> (none)

Commit message: fix router log module
Connections:
- net BTN_AC is gone; now on net X_ACT/FB_M1: U1.35 (PB14)
- net FB_M4 is gone; now on net X_ACT/FB_M1: U1.27 (PB1)
- net LED_DRY_GLASS_DRV is gone; now on net X_ACT/FB_M1: U1.3 (PC14)
- net LED_FACE_DRV is gone; now on net X_ACT/FB_M1: U1.55 (PB3)
- net M4_IN1 is gone; now on net X_ACT/FB_M1: U1.59 (PB7)
- net M4_IN2 is gone; now on net X_ACT/FB_M1: U1.2 (PC13)
- net M_FAN_CTL is gone; now on net X_ACT/FB_M1: U1.11 (PC3)
- net TEMP_SET_ADC is gone; now on net X_ACT/FB_M1: U1.14 (PA0)
- net AC_REQ_OUT renamed X_ACT/FB_M1
- net X_ACT/FB_M1: no longer C10.2, C21.2, C5.2, C6.2, C7.2, C8.2, C9.2, J2.3 (Pin_3), J2.4 (Pin_4), R2.2, U1.10 (PC2), U1.12 (VSSA), U1.18 (VSS), U1.26 (PB0), U1.31 (VSS), U1.4 (PC15), U1.47 (VSS), U1.49 (PA14), U1.57 (PB5), U1.62 (PB9), U1.63 (VSS)
- new net CAN_TX: U1.62 (PB9)
- new net FB_M3: U1.26 (PB0)
- new net GND: C5.2, U1.18 (VSS), U1.31 (VSS), U1.47 (VSS), U1.63 (VSS)
- new net LED_AC_DRV: U1.4 (PC15)
- new net LED_RECIRC_DRV: U1.10 (PC2)
- new net M3_IN1: U1.57 (PB5)
- new net SWCLK: J2.3 (Pin_3), U1.49 (PA14)

Commit message: fix router map cell no more mark for pins
Connections:
- net BTN_RECIRC is gone; now on net X_ACT/FB_M1: U1.36 (PB15)
- net CAN_TX is gone; now on net X_ACT/FB_M1: U1.62 (PB9)
- net FB_M3 is gone; now on net X_ACT/FB_M1: U1.26 (PB0)
- net GND is gone; now on net X_ACT/FB_M1: C5.2, U1.18 (VSS), U1.31 (VSS), U1.47 (VSS), U1.63 (VSS)
- net ILLUM_SENSE is gone; now on net X_ACT/FB_M1: U1.8 (PC0)
- net LED_DEFROST_GLASS_DRV is gone; now on net X_ACT/FB_M1: U1.50 (PA15)
- net LED_RECIRC_DRV is gone; now on net X_ACT/FB_M1: U1.10 (PC2)
- net M3_IN1 is gone; now on net X_ACT/FB_M1: U1.57 (PB5)
- net X_ACT/FB_M1: now also C10.2, C21.2, C6.2, C7.2, C8.2, C9.2, J2.4 (Pin_4), R2.2, U1.12 (VSSA); no longer U1.27 (PB1), U1.28 (PB2), U1.30 (PB11)
- new net AC_CTL: U1.28 (PB2)
- new net BTN_FACE: U1.30 (PB11)
- new net FB_M4: U1.27 (PB1)
Other:
- sheet X_ACT: file sheets/actuators.kicad_sch -> actuators.kicad_sch
- sheet X_BACKLIGHT: file sheets/backlight.kicad_sch -> backlight.kicad_sch
- sheet X_CAN: file sheets/can_bus.kicad_sch -> can_bus.kicad_sch
- sheet X_OUT: file sheets/power_outputs.kicad_sch -> power_outputs.kicad_sch
- sheet X_PWR: file sheets/power_supply.kicad_sch -> power_supply.kicad_sch
- sheet X_SEN_CABIN: file sheets/cabin_sensor.kicad_sch -> cabin_sensor.kicad_sch
- sheet X_SEN_COND: file sheets/condensate_sensor.kicad_sch -> condensate_sensor.kicad_sch
- sheet X_SEN_HEAT: file sheets/heating_sensor.kicad_sch -> heating_sensor.kicad_sch
- sheet X_SEN_SOLAR: file sheets/solar_sensor.kicad_sch -> solar_sensor.kicad_sch
- sheet X_UI: file sheets/user_interface.kicad_sch -> user_interface.kicad_sch

Commit message: рефакторинг проекта и начала прогона тестов
Connections:
- net FB_M4 is gone; now on net GND: U1.27 (PB1)
- net LED_AC_DRV is gone; now on net GND: U1.4 (PC15)
- net AC_CTL renamed GND
- net GND: now also C10.1, C10.2, C21.1, C21.2, C5.1, C5.2, C6.1, C6.2, C7.1, C7.2, C8.1, C8.2, C9.1, C9.2, FB1.1, FB1.2, J2.1 (Pin_1), J2.2 (Pin_2), J2.4 (Pin_4), R1.1, R1.2, R2.1, R2.2, U1.1 (VBAT), U1.12 (VSSA), U1.13 (VDDA), U1.14 (PA0), U1.15 (PA1), U1.16 (PA2), U1.17 (PA3), U1.18 (VSS), U1.19 (VDD), U1.2 (PC13), U1.20 (PA4), U1.22 (PA6), U1.23 (PA7), U1.26 (PB0), U1.3 (PC14), U1.31 (VSS), U1.32 (VDD), U1.41 (PA8), U1.42 (PA9), U1.43 (PA10), U1.44 (PA11), U1.45 (PA12), U1.46 (PA13), U1.47 (VSS), U1.48 (VDD), U1.50 (PA15), U1.55 (PB3), U1.56 (PB4), U1.57 (PB5), U1.58 (PB6), U1.59 (PB7), U1.60 (BOOT0), U1.61 (PB8), U1.62 (PB9), U1.63 (VSS), U1.64 (VDD), U1.7 (NRST)
- removed net X_ACT/FB_M1: C10.1, C10.2, C21.1, C21.2, C5.1, C5.2, C6.1, C6.2, C7.1, C7.2, C8.1, C8.2, C9.1, C9.2, FB1.1, FB1.2, J2.1 (Pin_1), J2.2 (Pin_2), J2.4 (Pin_4), R1.1, R1.2, R2.1, R2.2, U1.1 (VBAT), U1.10 (PC2), U1.11 (PC3), U1.12 (VSSA), U1.13 (VDDA), U1.14 (PA0), U1.15 (PA1), U1.16 (PA2), U1.17 (PA3), U1.18 (VSS), U1.19 (VDD), U1.2 (PC13), U1.20 (PA4), U1.21 (PA5), U1.22 (PA6), U1.23 (PA7), U1.26 (PB0), U1.29 (PB10), U1.3 (PC14), U1.31 (VSS), U1.32 (VDD), U1.33 (PB12), U1.34 (PB13), U1.35 (PB14), U1.36 (PB15), U1.41 (PA8), U1.42 (PA9), U1.43 (PA10), U1.44 (PA11), U1.45 (PA12), U1.46 (PA13), U1.47 (VSS), U1.48 (VDD), U1.50 (PA15), U1.55 (PB3), U1.56 (PB4), U1.57 (PB5), U1.58 (PB6), U1.59 (PB7), U1.60 (BOOT0), U1.61 (PB8), U1.62 (PB9), U1.63 (VSS), U1.64 (VDD), U1.7 (NRST), U1.8 (PC0)
- new net BTN_AC: U1.35 (PB14)
- new net BTN_DEFROST_GLASS: U1.29 (PB10)
- new net BTN_DRY_GLASS: U1.34 (PB13)
- new net BTN_FEET: U1.33 (PB12)
- new net BTN_RECIRC: U1.36 (PB15)
- new net COND_ADC: U1.21 (PA5)
- new net ILLUM_SENSE: U1.8 (PC0)
- new net LED_RECIRC_DRV: U1.10 (PC2)
- new net M_FAN_CTL: U1.11 (PC3)
Other:
- removed sheet X_ACT
- added sheet X_M1 (actuator_channel.kicad_sch)
- added sheet X_M2 (actuator_channel.kicad_sch)
- added sheet X_M3 (actuator_channel.kicad_sch)
- added sheet X_M4 (actuator_channel.kicad_sch)
- sheet X_UI ports: added GALLET_POS_1, GALLET_POS_2, GALLET_POS_3, GALLET_POS_4; removed none

Commit message: fix writer
Connections:
- net GND: no longer C10.1, C21.1, C5.1, C6.1, C7.1, C8.1, C9.1, FB1.1, FB1.2, J2.1 (Pin_1), J2.2 (Pin_2), R1.1, R1.2, R2.1, U1.1 (VBAT), U1.13 (VDDA), U1.14 (PA0), U1.15 (PA1), U1.16 (PA2), U1.17 (PA3), U1.19 (VDD), U1.2 (PC13), U1.20 (PA4), U1.22 (PA6), U1.23 (PA7), U1.26 (PB0), U1.27 (PB1), U1.28 (PB2), U1.3 (PC14), U1.32 (VDD), U1.4 (PC15), U1.41 (PA8), U1.42 (PA9), U1.43 (PA10), U1.44 (PA11), U1.45 (PA12), U1.46 (PA13), U1.48 (VDD), U1.50 (PA15), U1.55 (PB3), U1.56 (PB4), U1.57 (PB5), U1.58 (PB6), U1.59 (PB7), U1.60 (BOOT0), U1.61 (PB8), U1.62 (PB9), U1.64 (VDD), U1.7 (NRST)
- new net: C21.1, R1.2, U1.7 (NRST)
- new net: R2.1, U1.60 (BOOT0)
- new net X_CAN/CAN_RX: U1.61 (PB8)
- new net X_CAN/CAN_TX: U1.62 (PB9)
- new net X_M1/FB: U1.22 (PA6)
- new net X_M1/IN1: U1.42 (PA9), U1.43 (PA10)
- new net X_M2/FB: U1.23 (PA7)
- new net X_M2/IN1: U1.44 (PA11), U1.45 (PA12)
- new net X_M3/FB: U1.26 (PB0), U1.27 (PB1)
- new net X_M3/IN1: U1.57 (PB5), U1.58 (PB6)
- new net X_M4/IN1: U1.2 (PC13), U1.59 (PB7)
- new net X_OUT/AC_CTL: U1.28 (PB2)
- new net X_OUT/FAN_PWM_CTL: U1.41 (PA8)
- new net X_PWR/VCC_3V3: C5.1, C6.1, C7.1, C8.1, C9.1, FB1.1, J2.1 (Pin_1), R1.1, U1.1 (VBAT), U1.19 (VDD), U1.32 (VDD), U1.4 (PC15), U1.48 (VDD), U1.64 (VDD)
- new net X_SEN_CABIN/NTC_CABIN: U1.16 (PA2)
- new net X_SEN_HEAT/NTC_HEAT: U1.17 (PA3)
- new net X_SEN_SOLAR/SOLAR_ADC: U1.20 (PA4)
- new net X_UI/FAN_SEL_ADC: U1.15 (PA1)
- new net X_UI/LED_DEFROST_GLASS_DRV: C10.1, FB1.2, J2.2 (Pin_2), U1.13 (VDDA), U1.46 (PA13), U1.50 (PA15)
- new net X_UI/LED_DRY_GLASS_DRV: U1.3 (PC14)
- new net X_UI/LED_FACE_DRV: U1.55 (PB3)
- new net X_UI/LED_FEET_DRV: U1.56 (PB4)
- new net X_UI/TEMP_SET_ADC: U1.14 (PA0)
