File: climate_control_niva_travel.kicad_sch (KiCad schematic)
At the start: 12 parts, among them J2 SWD debug 1x04, U1 STM32G071RBT6

Commit message: refactoring
Parts:
- removed U1: STM32G071RBT6, symbol MyMCU:STM32G071RBT6
- added U1: STM32G071RBT6, symbol projectLib:STM32G071RBT6
Connections:
- net AC_CTL: now also U1.29 (PB2)
- net BTN_AC: now also U1.34 (PB14)
- net BTN_DEFROST_GLASS: now also U1.30 (PB10)
- net BTN_DRY_GLASS: now also U1.33 (PB13)
- net BTN_FACE: now also U1.31 (PB11)
- net BTN_FEET: now also U1.32 (PB12)
- net BTN_RECIRC: now also U1.35 (PB15)
- net CAN_RX: now also U1.62 (PB8)
- net CAN_TX: now also U1.63 (PB9)
- net COND_ADC: now also U1.22 (PA5)
- net FAN_PWM_CTL: now also U1.36 (PA8)
- net FAN_SEL_ADC: now also U1.16 (PC3), U1.18 (PA1)
- net FB_M1: now also U1.23 (PA6)
- net FB_M2: now also U1.24 (PA7)
- net FB_M3: now also U1.27 (PB0)
- net FB_M4: now also U1.28 (PB1)
- net GND: now also U1.9 (VSS/VSSA)
- net ILLUM_SENSE: now also U1.13 (PC0), U1.21 (PA4)
- net LED_AC_DRV: now also U1.5 (PC15-OSC32_OUT)
- net LED_DEFROST_GLASS_DRV: now also U1.47 (PA15)
- net LED_DRY_GLASS_DRV: now also U1.4 (PC14-OSC32_IN)
- net LED_FACE_DRV: now also U1.57 (PB3)
- net LED_FEET_DRV: now also U1.58 (PB4)
- net LED_RECIRC_DRV: now also U1.15 (PC2)
- net M1_IN1: now also U1.37 (PA9)
- net M1_IN2: now also U1.42 (PA10)
- net M2_IN1: now also U1.43 (PA11[PA9])
- net M2_IN2: now also U1.44 (PA12[PA10])
- net M3_IN1: now also U1.59 (PB5)
- net M3_IN2: now also U1.60 (PB6)
- net M4_IN1: now also U1.61 (PB7)
- net M4_IN2: now also U1.3 (PC13)
- net NRST: now also U1.12 (PF2-NRST)
- net NTC_CABIN: now also U1.19 (PA2)
- net NTC_HEAT: now also U1.20 (PA3)
- net SWCLK: now also U1.46 (PA14-BOOT0)
- net SWDIO: now also U1.45 (PA13)
- net TEMP_SET_ADC: now also U1.17 (PA0)
- net VCC_3V3: now also U1.6 (VBAT), U1.8 (VDD/VDDA)
- net VDDA_3V3: now also U1.7 (VREF+)

Commit message: multiInstance path fix
Parts:
- added J1: Разъём к автомобилю 2x16 (32 конт.), symbol Connector_Generic:Conn_02x16_Odd_Even
Connections:
- net LED_DRY_GLASS_DRV is gone; now on net LED_AC_DRV: U1.4 (PC14-OSC32_IN)
- net M4_IN2 is gone; now on net FB_M2: U1.3 (PC13)
- net AC_REQ_OUT: now also J1.24 (Pin_24)
- net CANH: now also J1.25 (Pin_25)
- net CANL: now also J1.26 (Pin_26)
- net COND_IN_RAW: now also J1.21 (Pin_21)
- net FAN_SEL_ADC: no longer U1.16 (PC3)
- net FB_M1_RAW: now also J1.7 (Pin_7)
- net FB_M2: now also U1.21 (PA4)
- net FB_M2_RAW: now also J1.10 (Pin_10)
- net FB_M3_RAW: now also J1.13 (Pin_13)
- net FB_M4_RAW: now also J1.16 (Pin_16)
- net GND: now also J1.18 (Pin_18), J1.3 (Pin_3), J1.4 (Pin_4)
- net HEAT_FAN_PWM_CTL: now also J1.23 (Pin_23)
- net ILLUM_IN_RAW: now also J1.22 (Pin_22)
- net ILLUM_SENSE: no longer U1.21 (PA4)
- net MOTOR_1_A: now also J1.5 (Pin_5)
- net MOTOR_1_B: now also J1.6 (Pin_6)
- net MOTOR_2_A: now also J1.8 (Pin_8)
- net MOTOR_2_B: now also J1.9 (Pin_9)
- net MOTOR_3_A: now also J1.11 (Pin_11)
- net MOTOR_3_B: now also J1.12 (Pin_12)
- net MOTOR_4_A: now also J1.14 (Pin_14)
- net MOTOR_4_B: now also J1.15 (Pin_15)
- net NTC_HEAT_W: now also J1.19 (Pin_19)
- net SOLAR_IN_RAW: now also J1.20 (Pin_20)
- new net M_FAN_CTL: U1.16 (PC3)
- new net V5_SENS: J1.17 (Pin_17)
- new net VBAT_IN: J1.1 (Pin_1), J1.2 (Pin_2)
Other:
- sheet X_POWER_SUPPLY ports: added V5_SENS, VBAT_IN; removed AC_REQ_OUT, CANH, CANL, COND_IN_RAW, FB_M1_RAW, FB_M2_RAW, FB_M3_RAW, FB_M4_RAW, HEAT_FAN_PWM_CTL, ILLUM_IN_RAW, MOTOR_1_A, MOTOR_1_B, MOTOR_2_A, MOTOR_2_B, MOTOR_3_A, MOTOR_3_B, MOTOR_4_A, MOTOR_4_B, NTC_HEAT_W, SOLAR_IN_RAW

Commit message: e2e tests added
Connections:
- net ILLUM_SENSE is gone; now on net FB_M2: U1.13 (PC0)
- net M_FAN_CTL is gone; now on net FAN_SEL_ADC: U1.16 (PC3)
- net FB_M2: no longer U1.21 (PA4), U1.3 (PC13)
- net LED_AC_DRV: no longer U1.4 (PC14-OSC32_IN)
- new net LED_DRY_GLASS_DRV: U1.4 (PC14-OSC32_IN)
- new net M4_IN2: U1.3 (PC13)
- new net SOLAR_ADC: U1.21 (PA4)
