File: can_bus.kicad_sch (KiCad schematic)
At the start: 1 part, among them U8 MCP2562-E-SN

Commit message: fix
Changed lines of the file:
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@@
 				(instances
 			(project "climate_control_niva_travel"
-				(path "/a20a8d43-2e18-4318-8ef3-7f434a470dab/0b9c7715-47ab-423b-a493-835c78427256"(reference "U0808") (unit 1) )
+				(path "/b4e4bdad-5656-40b1-b824-e2f3c68d6f72"(reference "U8") (unit 1) )
+				(path "/aece091b-8e26-4b21-9786-1b0efc647a51/71abb4ed-6c29-4c3b-b1db-d27c1ec5286d"(reference "U0808") (unit 1) )
 			)
 		)
@@
 	(wire
 		(pts
-			(xy 16.51 12.7) (xy 19.05 12.7)
-		)
-		(stroke
-			(width 0)
-			(type default)
-		)
-	)
-	(wire
-		(pts
-			(xy 19.05 12.7) (xy 19.05 11.43)
+			(xy 16.51 12.7) (xy 17.78 12.7)
+		)
+		(stroke
+			(width 0)
+			(type default)
+		)
+	)
+	(wire
+		(pts
+			(xy 17.78 12.7) (xy 17.78 11.43)
 		)
 		(stroke
@@
 	)
 	(junction
-		(at 19.05 11.43)
+		(at 17.78 11.43)
 		(diameter 0.0000)
 		(color 0 0 0 0)
